File: Project/LeSTMovoz revision 2.kicad_pcb (KiCad board)
At the start: 2 copper layers, 242.9 x 76.2 mm, 121 parts, among them J1 USB_C_Receptacle_USB2.0, SW1 SKQGABE010, U1 STM32F072RBTx, U2 L78L33_TO92, U3 74AHCT1G125

Commit message: revision wip
Parts:
- D1, D10, D11, D12, D13, D14, D15, D16, D17, D18, D19, D2, D20, D21, D22, D23, D24, D25, D26, D27, D28, D29, D3, D30, D31, D32, D33, D34, D35, D36, D37, D38, D39, D4, D40, D5, D6, D7, D8, D9: footprint kbd:D3_TH_SMD_v2 -> kbd:D3_TH_SMD_v3
- MX1, MX10, MX11, MX12, MX13, MX14, MX15, MX16, MX17, MX18, MX19, MX2, MX20, MX21, MX22, MX23, MX24, MX25, MX26, MX27, MX28, MX29, MX3, MX30, MX31, MX32, MX33, MX34, MX35, MX36, MX37, MX38, MX39, MX4, MX40, MX41, MX42, MX5, MX6, MX7, MX8, MX9: footprint PCM_marbastlib-mx:SW_MX_1u -> MX_Alps_Hybrid:MX-Alps-Hybrid-1U
- SW1: value SKQGABE010 -> boot; footprint PCM_marbastlib-various:SW_SPST_SKQG_WithStem -> Button_Switch_THT:SW_PUSH_6mm_H4.3mm
- SW2: renamed from RST1; value SW_SPST -> reset; footprint PCM_marbastlib-various:SW_SPST_SKQG_WithStem -> Button_Switch_THT:SW_PUSH_6mm_H4.3mm
- moved SW1 4.45 mm to (142.6, 94.3)
- moved SW2 3.56 mm to (148.0, 89.8)
- renumbered C9 to C10, C10 to C11, C12 to C3, C3 to C4, C4 to C5, C5 to C6, C6 to C7, C7 to C8, C8 to C9, D44 to D41, D45 to D42, D41 to D43, D43 to D44, D42 to D45, R4 to R1, R5 to R2, R6 to R3, R7 to R4
Routing:
- net ROW2: track 158.6 -> 170.1 mm
- net ROW3: track 119.4 -> 130.5 mm
- net ROW1: track 196.2 -> 201.0 mm
- net ROW0: track 235.6 -> 239.2 mm
- net Net-(D22-A): track 99.5 -> 100.6 mm
- net Net-(D23-A): track 85.8 -> 86.9 mm
- net Net-(D25-A): track 49.2 -> 50.3 mm
- net Net-(D24-A): track 63.2 -> 64.4 mm
- net Net-(D5-A): track 48.0 -> 49.1 mm
- net Net-(D2-A): track 99.1 -> 100.2 mm
- net Net-(D1-A): track 120.9 -> 122.0 mm
- net Net-(D21-A): track 119.8 -> 120.8 mm
- net Net-(D4-A): track 62.6 -> 63.7 mm
- net Net-(D3-A): track 81.5 -> 82.5 mm
- net NRST: track 25.3 -> 26.1 mm
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Other:
- board text added: "USB here"
- board text removed: "USB"
