File: Project/LeSTMovoz revision 2.kicad_pcb (KiCad board)
At the start: 2 copper layers, 242.9 x 76.2 mm, 123 parts, among them J1 USB_C_Receptacle_USB2.0, SW1 boot, SW2 reset, U1 STM32F072RBTx, U2 L78L33_TO92, U3 74AHCT1G125

Commit message: production files
Parts:
- removed the J1 at (247.1, 13.6)
Connections:
- R5 pad 1: unconnected-(R5-Pad1) -> RGB MCU
- R5 pad 2: unconnected-(R5-Pad2) -> RGBin
Routing:
- net +5V: track 66.2 -> 67.1 mm
