File: Project/LeSTMovoz revision 2.kicad_pcb (KiCad board)
At the start: 2 copper layers, 242.9 x 76.2 mm, 122 parts, among them J1 USB_C_Receptacle_USB2.0, SW1 boot, SW2 reset, U1 STM32F072RBTx, U2 L78L33_TO92, U3 74AHCT1G125

Commit message: production files cleaned up
Parts:
- removed R5: 5k1, Resistor_THT:R_Axial_DIN0204_L3.6mm_D1.6mm_P7.62mm_Horizontal
