File: Project/LeSTMovoz revision 2.kicad_sch (KiCad schematic)
At the start: 116 parts, among them J1 USB_C_Receptacle_USB2.0, SW1 SKQGABE010, U1 STM32F072RBTx, U2 L78L33_TO92, U3 74AHCT1G125

Commit message: revison work
Parts:
- removed D42, D43: 3.6V, Diode_THT:D_DO-35_SOD27_P7.62mm_Horizontal, symbol lumberjack-rescue:D_Schottky_Small_ALT-Device
- removed R1: 1.5k, Resistor_THT:R_Axial_DIN0204_L3.6mm_D1.6mm_P7.62mm_Horizontal, symbol Device:R_Small
- removed R2, R3: 75R, Resistor_THT:R_Axial_DIN0204_L3.6mm_D1.6mm_P7.62mm_Horizontal, symbol Device:R_Small
- added D44, D45: 3.6V, Diode_THT:D_DO-35_SOD27_P7.62mm_Horizontal, symbol lumberjack-rescue:D_Schottky_Small_ALT-Device
- added R5: 5k1, Resistor_THT:R_Axial_DIN0204_L3.6mm_D1.6mm_P7.62mm_Horizontal, symbol Device:R_Small
- D1, D10, D11, D12, D13, D14, D15, D16, D17, D18, D19, D2, D20, D21, D22, D23, D24, D25, D26, D27, D28, D29, D3, D30, D31, D32, D33, D34, D35, D36, D37, D38, D39, D4, D40, D5, D6, D7, D8, D9: footprint kbd:D3_TH_SMD_v2 -> kbd:D3_TH_SMD_v3
- J1: footprint Connector_USB:USB_C_Receptacle_GCT_USB4085 -> PCM_marbastlib-various:USB_C_Receptacle_HRO_TYPE-C-31-M-12
- MX1, MX10, MX11, MX12, MX13, MX14, MX15, MX16, MX17, MX18, MX19, MX2, MX20, MX21, MX22, MX23, MX24, MX25, MX26, MX27, MX28, MX29, MX3, MX30, MX31, MX32, MX33, MX34, MX35, MX36, MX37, MX38, MX39, MX4, MX40, MX41, MX42, MX5, MX6, MX7, MX8, MX9: footprint PCM_marbastlib-mx:SW_MX_1u -> MX_Alps_Hybrid:MX-Alps-Hybrid-1U
- SW1: value SKQGABE010 -> boot; footprint PCM_marbastlib-various:SW_SPST_SKQG_WithStem -> Button_Switch_THT:SW_PUSH_6mm_H4.3mm
- SW2: renamed from RST1; value SW_SPST -> reset; footprint PCM_marbastlib-various:SW_SPST_SKQG_WithStem -> Button_Switch_THT:SW_PUSH_6mm_H4.3mm
- renumbered C9 to C10, C10 to C11, C12 to C3, C3 to C4, C4 to C5, C5 to C6, C6 to C7, C7 to C8, C8 to C9, D44 to D41, D45 to D42, D41 to D43, R4 to R1, R5 to R2, R6 to R3, R7 to R4
Connections:
- net D_USB_N is gone; now on net D_N: J1.A7 (D-), J1.B7 (D-)
- net D_USB_P is gone; now on net D_P: J1.A6 (D+), J1.B6 (D+)
- net D_N: now also D45.1 (K)
- net D_P: now also D44.1 (K)
- net GND: now also D44.2 (A), D45.2 (A)
- net RGB MCU: now also R5.1
- net RGBin: now also R5.2
Other:
- note added: "RGB leds"
- note added: "basic esd"
- note removed: "ESD"
- moved on the sheet: C3, D41, D42, S3, S4, U3
