File: Project/LeSTMovoz revision 2.kicad_sch (KiCad schematic)
At the start: 114 parts, among them J1 USB_C_Receptacle_USB2.0, SW1 boot, SW2 reset, U1 STM32F072RBTx, U2 L78L33_TO92, U3 74AHCT1G125

Commit message: production files cleaned up
Parts:
- R5: now not fitted; now left out of the parts list
Changed lines of the file:
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@@
 (kicad_sch
-	(version 20231120)
+	(version 20250114)
 	(generator "eeschema")
-	(generator_version "8.0")
+	(generator_version "9.0")
 	(paper "A4")
+	(rectangle
+		(start 12.7 118.745)
+		(end 69.215 196.85)
+		(stroke
+			(width 0)
+			(type default)
+		)
+		(fill
+			(type none)
+		)
+	)
+	(rectangle
+		(start 69.85 145.415)
+		(end 130.81 170.815)
+		(stroke
+			(width 0)
+			(type default)
+		)
+		(fill
+			(type none)
+		)
+	)
+	(rectangle
+		(start 106.045 118.745)
+		(end 140.335 144.78)
+		(stroke
+			(width 0)
+			(type default)
+		)
+		(fill
+			(type none)
+		)
+	)
+	(rectangle
+		(start 186.055 118.745)
+		(end 243.205 146.685)
+		(stroke
+			(width 0)
+			(type default)
+		)
+		(fill
+			(type none)
+		)
+	)
+	(rectangle
+		(start 69.85 118.745)
+		(end 105.41 144.78)
+		(stroke
+			(width 0)
+			(type default)
+		)
+		(fill
+			(type none)
+		)
+	)
+	(rectangle
+		(start 69.85 171.45)
+		(end 147.955 196.85)
+		(stroke
+			(width 0)
+			(type default)
+		)
+		(fill
+			(type none)
+		)
+	)
+	(rectangle
+		(start 140.97 118.745)
+		(end 185.42 150.495)
+		(stroke
+			(width 0)
+			(type default)
+		)
+		(fill
+			(type none)
+		)
+	)
+	(text "RGB leds"
+		(exclude_from_sim no)
+		(at 186.69 123.19 0)
+		(effects
+			(font
+				(size 2 2)
+			)
+			(justify left bottom)
+		)
+	)
+	(text "RGB logic shifter"
+		(exclude_from_sim no)
+		(at 158.75 149.225 0)
+		(effects
+			(font
+				(size 2 2)
+			)
+			(justify left bottom)
+		)
+	)
+	(text "capacitors"
+		(exclude_from_sim no)
+		(at 71.12 173.99 0)
+		(effects
+			(font
+				(size 1.27 1.27)
+			)
+			(justify left bottom)
+		)
+	)
+	(text "boot&nrst"
+		(exclude_from_sim no)
+		(at 71.12 147.955 0)
+		(effects
+			(font
+				(size 1.27 1.27)
+			)
+			(justify left bottom)
+		)
+	)
+	(text "3.3V LDO"
+		(exclude_from_sim no)
+		(at 71.755 121.92 0)
+		(effects
+			(font
+				(size 1.27 1.27)
+			)
+			(justify left bottom)
+		)
+	)
+	(text "USB"
+		(exclude_from_sim no)
+		(at 13.97 121.285 0)
+		(effects
+			(font
+				(size 1.27 1.27)
+			)
+			(justify left bottom)
+		)
+	)
+	(text "basic esd"
+		(exclude_from_sim no)
+		(at 106.68 121.285 0)
+		(effects
+			(font
+				(size 1.27 1.27)
+			)
+			(justify left bottom)
+		)
+	)
 	(junction
 		(at 226.06 92.075)
@@
 		)
 	)
-	(rectangle
-		(start 12.7 118.745)
-		(end 69.215 196.85)
-		(stroke
-			(width 0)
-			(type default)
-		)
-		(fill
-			(type none)
-		)
-	)
-	(rectangle
-		(start 69.85 145.415)
-		(end 130.81 170.815)
-		(stroke
-			(width 0)
-			(type default)
-		)
-		(fill
-			(type none)
-		)
-	)
-	(rectangle
-		(start 106.045 118.745)
-		(end 140.335 144.78)
-		(stroke
-			(width 0)
-			(type default)
-		)
-		(fill
-			(type none)
-		)
-	)
-	(rectangle
-		(start 186.055 118.745)
-		(end 243.205 146.685)
-		(stroke
-			(width 0)
-			(type default)
-		)
-		(fill
-			(type none)
-		)
-	)
-	(rectangle
-		(start 69.85 118.745)
-		(end 105.41 144.78)
-		(stroke
-			(width 0)
-			(type default)
-		)
-		(fill
-			(type none)
-		)
-	)
-	(rectangle
-		(start 69.85 171.45)
-		(end 147.955 196.85)
-		(stroke
-			(width 0)
-			(type default)
-		)
-		(fill
-			(type none)
-		)
-	)
-	(rectangle
-		(start 140.97 118.745)
-		(end 185.42 150.495)
-		(stroke
-			(width 0)
-			(type default)
-		)
-		(fill
-			(type none)
-		)
-	)
-	(text "RGB leds"
-		(exclude_from_sim no)
-		(at 186.69 123.19 0)
-		(effects
-			(font
-				(size 2 2)
-			)
-			(justify left bottom)
-		)
-	)
-	(text "RGB logic shifter"
-		(exclude_from_sim no)
-		(at 158.75 149.225 0)
-		(effects
-			(font
-				(size 2 2)
-			)
-			(justify left bottom)
-		)
-	)
-	(text "capacitors"
-		(exclude_from_sim no)
-		(at 71.12 173.99 0)
-		(effects
-			(font
-				(size 1.27 1.27)
-			)
-			(justify left bottom)
-		)
-	)
-	(text "boot&nrst"
-		(exclude_from_sim no)
-		(at 71.12 147.955 0)
-		(effects
-			(font
-				(size 1.27 1.27)
-			)
-			(justify left bottom)
-		)
-	)
-	(text "3.3V LDO"
-		(exclude_from_sim no)
-		(at 71.755 121.92 0)
-		(effects
-			(font
-				(size 1.27 1.27)
-			)
-			(justify left bottom)
-		)
-	)
-	(text "USB"
-		(exclude_from_sim no)
-		(at 13.97 121.285 0)
-		(effects
-			(font
-				(size 1.27 1.27)
-			)
-			(justify left bottom)
-		)
-	)
-	(text "basic esd"
-		(exclude_from_sim no)
-		(at 106.68 121.285 0)
-		(effects
-			(font
-				(size 1.27 1.27)
-			)
-			(justify left bottom)
-		)
-	)
 	(label "CC1"
 		(at 43.18 153.035 0)
@@
 		(at 157.48 113.03 90)
 		(unit 1)
-		(exclude_from_sim no)
-		(in_bom yes)
-		(on_board yes)
-		(dnp no)
+		(exclude_from_sim yes)
+		(in_bom no)
+		(on_board no)
+		(dnp yes)
 		(property "Reference" "R5"
 			(at 157.48 113.03 90)
@@
 		)
 	)
+	(embedded_fonts no)
 )
