File: Project/LeSTMovoz revision 2 rotaries.kicad_pcb (KiCad board)
At the start: 2 copper layers, 242.9 x 76.2 mm, 121 parts, among them J1 USB_C_Receptacle_USB2.0, SW1 boot, SW2 reset, U1 STM32F072RBTx, U2 L78L33_TO92, U3 74AHCT1G125

Commit message: revision wip
Parts:
- added SW3: RotaryEncoder_Switch, PCM_marbastlib-various:ROT_Alps_EC11E-Switch, F.Cu at (33.3, 33.3)
- added SW4: RotaryEncoder_Switch, PCM_marbastlib-various:ROT_Alps_EC11E-Switch, F.Cu at (257.2, 33.3)
- moved C11 0.37 mm to (138.9, 62.0)
- moved C6 0.37 mm to (136.5, 62.0)
- moved C9 0.37 mm to (152.4, 62.0)
- moved G*** 0.37 mm to (145.3, 59.2)
Connections:
- net Net-(D1-A) renamed r_enc1
- net Net-(D10-A) renamed r_enc2
- U1 pad 27: unconnected-(U1-PB1-Pad27) -> ENC_D
- U1 pad 28: unconnected-(U1-PB2-Pad28) -> ENC_C
- U1 pad 53: unconnected-(U1-PC12-Pad53) -> ENC_B
- U1 pad 54: unconnected-(U1-PD2-Pad54) -> ENC_A
Routing:
- net ENC_A: track 0.00 -> 134.2 mm
- net ENC_D: track 0.00 -> 131.3 mm
- net ENC_C: track 0.00 -> 129.3 mm, vias 0 -> 2
- net ENC_B: track 0.00 -> 129.0 mm
- net r_enc1: track 122.0 -> 129.3 mm
- net COL0: track 180.0 -> 184.5 mm
- net COL9: track 172.9 -> 177.4 mm
- net +3V3: track 123.1 -> 126.5 mm
- net Net-(D5-A): track 49.1 -> 47.1 mm
- net Net-(D9-A): track 77.2 -> 79.2 mm, vias 0 -> 1
- net r_enc2: track 119.3 -> 121.1 mm
- net Net-(D4-A): track 63.7 -> 62.1 mm
- net Net-(D7-A): track 58.1 -> 56.7 mm
- net Net-(D6-A): track 42.6 -> 41.5 mm
- net Net-(D8-A): track 76.0 -> 74.9 mm
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Other:
- board text added: "ENC"
